File: kicad-global/Basic-DC-mixer.kicad_sch (KiCad schematic)
At the start: 37 parts, among them J1 In, J2 Power Input, J3 In, J4 InvOut, J5 Out, J6 In, J7 In, SW1 Mute, SW2 Mute, SW3 Mute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

Commit message: update mixer to v1.2, update repo organization
Parts:
- removed J1, J3, J6, J7: In, Synth:Thonkiconn, symbol Connector:AudioJack2_Switch
- removed J4: InvOut, Synth:Thonkiconn, symbol Connector:AudioJack2_Switch
- removed J5: Out, Synth:Thonkiconn, symbol Connector:AudioJack2_Switch
- added J1, J3, J6, J7: In, Kicad-perso:Thonkiconn, symbol Kicad-perso:AudioJack_Switch
- added J4: InvOut, Kicad-perso:Thonkiconn, symbol Kicad-perso:AudioJack_Switch
- added J5: Out, Kicad-perso:Thonkiconn, symbol Kicad-perso:AudioJack_Switch
- H1, H2, H3, H4: now left out of the parts list
- J2: footprint Connector_PinHeader_2.54mm:PinHeader_2x05_P2.54mm_Vertical -> Connector_IDC:IDC-Header_2x05_P2.54mm_Vertical
- SW1, SW2, SW3, SW4: footprint Synth:SW_DPDT_Toggle -> Kicad-perso:SW_DPDT_Toggle; Comments (none) -> DPDT On-ON
- Vol1, Vol2, Vol3, Vol4: footprint Synth:Pot-bourns-alpha -> Kicad-perso:Pot-bourns-alpha
Connections:
- net +12V: now also J2.10 (Pin_10), J2.9 (Pin_9); no longer J2.1 (Pin_1), J2.2 (Pin_2)
- net -12V: now also J2.1 (Pin_1), J2.2 (Pin_2); no longer J2.10 (Pin_10), J2.9 (Pin_9)
- net GND: now also Vol1.1, Vol2.1, Vol3.1, Vol4.1, J1.S, J3.S, J4.S, J5.S, J6.S, J7.S; no longer Vol1.3, Vol2.3, Vol3.3, Vol4.3
- net at R7.1, U1.1: now also J5.T
- net at R6.2, R8.1, U1.7: now also J4.T
- net at SW1.5 (B): now also J1.T
- net at SW3.6 (C): now also Vol3.3; no longer Vol3.1
- net at SW4.6 (C): now also Vol4.3; no longer Vol4.1
- net at SW3.5 (B): now also J6.T
- net at SW2.5 (B): now also J3.T
- net at SW2.6 (C): now also Vol2.3; no longer Vol2.1
- net at SW1.6 (C): now also Vol1.3; no longer Vol1.1
- net at SW4.5 (B): now also J7.T
- no-connect marks 20 -> 14
Other:
- company: (none) -> Bleep Sound
- title: (none) -> Active DC coupled mixer
